Commit message: Update HyA urdf, IK solver, fix DARE exceptions.

File: ct_models/urdf/HyA/HyA.urdf (robot description, URDF)
Before this commit: robot hya, 7 links, 6 joints
Links:
- added link hya_ee0
Joints:
- added joint hya_ee0_joint: type fixed, parent hya_wrist_fe_link, child hya_ee0, origin xyz=0.03 0 0, axis 0 0 0, limit lower=0 upper=0 effort=100 velocity=0.5
